File: FEAR-16 - Mainboard.kicad_pcb (KiCad board)
At the start: 4 copper layers, 224 x 395 mm, 344 parts, among them IC101 EK-TM4C123GXL, J101 Screw_5.08, J2501 Screw_5.08, P2101 USB-C, U101 FT232RL, U102 SN74LVC1G14DBV, U103 SN74LVC1G14DBV, U104 HCPL-2631, U105 HCPL-2631, U106 SN74LVC1G14DBV, U107 SN74LVC1G14DBV, U1101 DACx1408, U1301 ADS8568, U1401 ADP2370, U1402 uA7805, U2201 ADS8568, U2301 DACx1408, U2401 ADS8568, U2501 ADS8568

Commit message: FEAR-16 V2.2
PCB-Changes:
 - Added rudimentary "load-balancer" (not really a balancer, but should avoid the DC/DC from regulating against each other!)
 - Added optional GND-jumpers to the N/C pins of the shields
 - Modified amplification adjustment:
   -> Added a offset resistor in row to the trim-poti for amplification for finer amp-tuning
   -> Reduced trim-poti-value from 1Meg -> 50k (20x finer adjustment-range)
      Poti can in the range of:
      - 30k (min) for being able to reach the correct amplification
      - 50k (max) for having at least 20x finer tune-range and a bit of reserve, as 30k is pretty thight on tolerance

Misc.:
 - Added LICENSE.md
Parts:
- added JP1001: Opt. GND, Jumper:SolderJumper-2_P1.3mm_Open_RoundedPad1.0x1.5mm, F.Cu at (176.3, 338.0)
- added JP1002: Opt. GND, Jumper:SolderJumper-2_P1.3mm_Open_RoundedPad1.0x1.5mm, F.Cu at (176.3, 335.5)
- added JP1003: Opt. GND, Jumper:SolderJumper-2_P1.3mm_Open_RoundedPad1.0x1.5mm, F.Cu at (176.3, 332.9)
- added JP1004: Opt. GND, Jumper:SolderJumper-2_P1.3mm_Open_RoundedPad1.0x1.5mm, F.Cu at (176.3, 327.8)
- added JP1005: Opt. GND, Jumper:SolderJumper-2_P1.3mm_Open_RoundedPad1.0x1.5mm, F.Cu at (176.3, 322.8)
- added JP1201: Opt. GND, Jumper:SolderJumper-2_P1.3mm_Open_RoundedPad1.0x1.5mm, F.Cu at (176.3, 297.0)
- added JP1202: Opt. GND, Jumper:SolderJumper-2_P1.3mm_Open_RoundedPad1.0x1.5mm, F.Cu at (176.3, 294.5)
- added JP1203: Opt. GND, Jumper:SolderJumper-2_P1.3mm_Open_RoundedPad1.0x1.5mm, F.Cu at (176.3, 291.9)
- added JP1204: Opt. GND, Jumper:SolderJumper-2_P1.3mm_Open_RoundedPad1.0x1.5mm, F.Cu at (176.3, 286.8)
- added JP1205: Opt. GND, Jumper:SolderJumper-2_P1.3mm_Open_RoundedPad1.0x1.5mm, F.Cu at (176.3, 281.8)
- added JP1501: Opt. GND, Jumper:SolderJumper-2_P1.3mm_Open_RoundedPad1.0x1.5mm, F.Cu at (176.3, 256.0)
- added JP1502: Opt. GND, Jumper:SolderJumper-2_P1.3mm_Open_RoundedPad1.0x1.5mm, F.Cu at (176.3, 253.5)
- added JP1503: Opt. GND, Jumper:SolderJumper-2_P1.3mm_Open_RoundedPad1.0x1.5mm, F.Cu at (176.3, 250.9)
- added JP1504: Opt. GND, Jumper:SolderJumper-2_P1.3mm_Open_RoundedPad1.0x1.5mm, F.Cu at (176.3, 245.8)
- added JP1505: Opt. GND, Jumper:SolderJumper-2_P1.3mm_Open_RoundedPad1.0x1.5mm, F.Cu at (176.3, 240.8)
- added JP1601: Opt. GND, Jumper:SolderJumper-2_P1.3mm_Open_RoundedPad1.0x1.5mm, F.Cu at (176.3, 215.0)
- added JP1602: Opt. GND, Jumper:SolderJumper-2_P1.3mm_Open_RoundedPad1.0x1.5mm, F.Cu at (176.3, 212.5)
- added JP1603: Opt. GND, Jumper:SolderJumper-2_P1.3mm_Open_RoundedPad1.0x1.5mm, F.Cu at (176.3, 209.9)
- added JP1604: Opt. GND, Jumper:SolderJumper-2_P1.3mm_Open_RoundedPad1.0x1.5mm, F.Cu at (176.3, 204.8)
- added JP1605: Opt. GND, Jumper:SolderJumper-2_P1.3mm_Open_RoundedPad1.0x1.5mm, F.Cu at (176.3, 199.8)
- added JP1701: Opt. GND, Jumper:SolderJumper-2_P1.3mm_Open_RoundedPad1.0x1.5mm, F.Cu at (176.3, 174.0)
- added JP1702: Opt. GND, Jumper:SolderJumper-2_P1.3mm_Open_RoundedPad1.0x1.5mm, F.Cu at (176.3, 171.5)
- added JP1703: Opt. GND, Jumper:SolderJumper-2_P1.3mm_Open_RoundedPad1.0x1.5mm, F.Cu at (176.3, 168.9)
- added JP1704: Opt. GND, Jumper:SolderJumper-2_P1.3mm_Open_RoundedPad1.0x1.5mm, F.Cu at (176.3, 163.8)
- added JP1705: Opt. GND, Jumper:SolderJumper-2_P1.3mm_Open_RoundedPad1.0x1.5mm, F.Cu at (176.3, 158.8)
- added JP1801: Opt. GND, Jumper:SolderJumper-2_P1.3mm_Open_RoundedPad1.0x1.5mm, F.Cu at (47.7, 58.0)
- added JP1802: Opt. GND, Jumper:SolderJumper-2_P1.3mm_Open_RoundedPad1.0x1.5mm, F.Cu at (47.7, 60.5)
- added JP1803: Opt. GND, Jumper:SolderJumper-2_P1.3mm_Open_RoundedPad1.0x1.5mm, F.Cu at (47.7, 63.1)
- added JP1804: Opt. GND, Jumper:SolderJumper-2_P1.3mm_Open_RoundedPad1.0x1.5mm, F.Cu at (47.7, 68.2)
- added JP1805: Opt. GND, Jumper:SolderJumper-2_P1.3mm_Open_RoundedPad1.0x1.5mm, F.Cu at (47.7, 73.2)
- added JP1901: Opt. GND, Jumper:SolderJumper-2_P1.3mm_Open_RoundedPad1.0x1.5mm, F.Cu at (176.3, 133.0)
- added JP1902: Opt. GND, Jumper:SolderJumper-2_P1.3mm_Open_RoundedPad1.0x1.5mm, F.Cu at (176.3, 130.5)
- added JP1903: Opt. GND, Jumper:SolderJumper-2_P1.3mm_Open_RoundedPad1.0x1.5mm, F.Cu at (176.3, 127.9)
- added JP1904: Opt. GND, Jumper:SolderJumper-2_P1.3mm_Open_RoundedPad1.0x1.5mm, F.Cu at (176.3, 122.8)
- added JP1905: Opt. GND, Jumper:SolderJumper-2_P1.3mm_Open_RoundedPad1.0x1.5mm, F.Cu at (176.3, 117.8)
- added JP2001: Opt. GND, Jumper:SolderJumper-2_P1.3mm_Open_RoundedPad1.0x1.5mm, F.Cu at (176.3, 92.0)
- added JP2002: Opt. GND, Jumper:SolderJumper-2_P1.3mm_Open_RoundedPad1.0x1.5mm, F.Cu at (176.3, 89.5)
- added JP2003: Opt. GND, Jumper:SolderJumper-2_P1.3mm_Open_RoundedPad1.0x1.5mm, F.Cu at (176.3, 86.9)
- added JP2004: Opt. GND, Jumper:SolderJumper-2_P1.3mm_Open_RoundedPad1.0x1.5mm, F.Cu at (176.3, 81.8)
- added JP2005: Opt. GND, Jumper:SolderJumper-2_P1.3mm_Open_RoundedPad1.0x1.5mm, F.Cu at (176.3, 76.8)
- added JP201: Opt. GND, Jumper:SolderJumper-2_P1.3mm_Open_RoundedPad1.0x1.5mm, F.Cu at (47.7, 99.0)
- added JP202: Opt. GND, Jumper:SolderJumper-2_P1.3mm_Open_RoundedPad1.0x1.5mm, F.Cu at (47.7, 101.5)
- added JP203: Opt. GND, Jumper:SolderJumper-2_P1.3mm_Open_RoundedPad1.0x1.5mm, F.Cu at (47.7, 104.1)
- added JP204: Opt. GND, Jumper:SolderJumper-2_P1.3mm_Open_RoundedPad1.0x1.5mm, F.Cu at (47.7, 109.2)
- added JP205: Opt. GND, Jumper:SolderJumper-2_P1.3mm_Open_RoundedPad1.0x1.5mm, F.Cu at (47.7, 114.2)
- added JP301: Opt. GND, Jumper:SolderJumper-2_P1.3mm_Open_RoundedPad1.0x1.5mm, F.Cu at (47.7, 140.0)
- added JP302: Opt. GND, Jumper:SolderJumper-2_P1.3mm_Open_RoundedPad1.0x1.5mm, F.Cu at (47.7, 142.5)
- added JP303: Opt. GND, Jumper:SolderJumper-2_P1.3mm_Open_RoundedPad1.0x1.5mm, F.Cu at (47.7, 145.1)
- added JP304: Opt. GND, Jumper:SolderJumper-2_P1.3mm_Open_RoundedPad1.0x1.5mm, F.Cu at (47.7, 150.2)
- added JP305: Opt. GND, Jumper:SolderJumper-2_P1.3mm_Open_RoundedPad1.0x1.5mm, F.Cu at (47.7, 155.2)
- added JP401: Opt. GND, Jumper:SolderJumper-2_P1.3mm_Open_RoundedPad1.0x1.5mm, F.Cu at (47.7, 181.0)
- added JP402: Opt. GND, Jumper:SolderJumper-2_P1.3mm_Open_RoundedPad1.0x1.5mm, F.Cu at (47.7, 183.5)
- added JP403: Opt. GND, Jumper:SolderJumper-2_P1.3mm_Open_RoundedPad1.0x1.5mm, F.Cu at (47.7, 186.1)
- added JP404: Opt. GND, Jumper:SolderJumper-2_P1.3mm_Open_RoundedPad1.0x1.5mm, F.Cu at (47.7, 191.2)
- added JP405: Opt. GND, Jumper:SolderJumper-2_P1.3mm_Open_RoundedPad1.0x1.5mm, F.Cu at (47.7, 196.2)
- added JP501: Opt. GND, Jumper:SolderJumper-2_P1.3mm_Open_RoundedPad1.0x1.5mm, F.Cu at (47.7, 222.0)
- added JP502: Opt. GND, Jumper:SolderJumper-2_P1.3mm_Open_RoundedPad1.0x1.5mm, F.Cu at (47.7, 224.5)
- added JP503: Opt. GND, Jumper:SolderJumper-2_P1.3mm_Open_RoundedPad1.0x1.5mm, F.Cu at (47.7, 227.1)
- added JP504: Opt. GND, Jumper:SolderJumper-2_P1.3mm_Open_RoundedPad1.0x1.5mm, F.Cu at (47.7, 232.2)
- added JP505: Opt. GND, Jumper:SolderJumper-2_P1.3mm_Open_RoundedPad1.0x1.5mm, F.Cu at (47.7, 237.2)
- added JP601: Opt. GND, Jumper:SolderJumper-2_P1.3mm_Open_RoundedPad1.0x1.5mm, F.Cu at (47.7, 263.0)
- added JP602: Opt. GND, Jumper:SolderJumper-2_P1.3mm_Open_RoundedPad1.0x1.5mm, F.Cu at (47.7, 265.5)
- added JP603: Opt. GND, Jumper:SolderJumper-2_P1.3mm_Open_RoundedPad1.0x1.5mm, F.Cu at (47.7, 268.1)
- added JP604: Opt. GND, Jumper:SolderJumper-2_P1.3mm_Open_RoundedPad1.0x1.5mm, F.Cu at (47.7, 273.2)
- added JP605: Opt. GND, Jumper:SolderJumper-2_P1.3mm_Open_RoundedPad1.0x1.5mm, F.Cu at (47.7, 278.2)
- added JP701: Opt. GND, Jumper:SolderJumper-2_P1.3mm_Open_RoundedPad1.0x1.5mm, F.Cu at (47.7, 304.0)
- added JP702: Opt. GND, Jumper:SolderJumper-2_P1.3mm_Open_RoundedPad1.0x1.5mm, F.Cu at (47.7, 306.5)
- added JP703: Opt. GND, Jumper:SolderJumper-2_P1.3mm_Open_RoundedPad1.0x1.5mm, F.Cu at (47.7, 309.1)
- added JP704: Opt. GND, Jumper:SolderJumper-2_P1.3mm_Open_RoundedPad1.0x1.5mm, F.Cu at (47.7, 314.2)
- added JP705: Opt. GND, Jumper:SolderJumper-2_P1.3mm_Open_RoundedPad1.0x1.5mm, F.Cu at (47.7, 319.2)
- added JP801: Opt. GND, Jumper:SolderJumper-2_P1.3mm_Open_RoundedPad1.0x1.5mm, F.Cu at (47.7, 345.0)
- added JP802: Opt. GND, Jumper:SolderJumper-2_P1.3mm_Open_RoundedPad1.0x1.5mm, F.Cu at (47.7, 347.5)
- added JP803: Opt. GND, Jumper:SolderJumper-2_P1.3mm_Open_RoundedPad1.0x1.5mm, F.Cu at (47.7, 350.1)
- added JP804: Opt. GND, Jumper:SolderJumper-2_P1.3mm_Open_RoundedPad1.0x1.5mm, F.Cu at (47.7, 355.2)
- added JP805: Opt. GND, Jumper:SolderJumper-2_P1.3mm_Open_RoundedPad1.0x1.5mm, F.Cu at (47.7, 360.2)
- added JP901: Opt. GND, Jumper:SolderJumper-2_P1.3mm_Open_RoundedPad1.0x1.5mm, F.Cu at (176.3, 379.0)
- added JP902: Opt. GND, Jumper:SolderJumper-2_P1.3mm_Open_RoundedPad1.0x1.5mm, F.Cu at (176.3, 376.5)
- added JP903: Opt. GND, Jumper:SolderJumper-2_P1.3mm_Open_RoundedPad1.0x1.5mm, F.Cu at (176.3, 373.9)
- added JP904: Opt. GND, Jumper:SolderJumper-2_P1.3mm_Open_RoundedPad1.0x1.5mm, F.Cu at (176.3, 368.8)
- added JP905: Opt. GND, Jumper:SolderJumper-2_P1.3mm_Open_RoundedPad1.0x1.5mm, F.Cu at (176.3, 363.8)
Connections:
- Channel0 pad 10: unconnected-(Channel0-Pad10) -> Net-(JP1802-A)
- Channel0 pad 11: unconnected-(Channel0-Pad11) -> Net-(JP1803-A)
- Channel0 pad 13: unconnected-(Channel0-Pad13) -> Net-(JP1804-A)
- Channel0 pad 15: unconnected-(Channel0-Pad15) -> Net-(JP1805-A)
- Channel0 pad 9: unconnected-(Channel0-Pad9) -> Net-(JP1801-A)
- Channel1 pad 10: unconnected-(Channel1-Pad10) -> Net-(JP202-A)
- Channel1 pad 11: unconnected-(Channel1-Pad11) -> Net-(JP203-A)
- Channel1 pad 13: unconnected-(Channel1-Pad13) -> Net-(JP204-A)
- Channel1 pad 15: unconnected-(Channel1-Pad15) -> Net-(JP205-A)
- Channel1 pad 9: unconnected-(Channel1-Pad9) -> Net-(JP201-A)
- Channel10 pad 10: unconnected-(Channel10-Pad10) -> Net-(JP1202-A)
- Channel10 pad 11: unconnected-(Channel10-Pad11) -> Net-(JP1203-A)
- Channel10 pad 13: unconnected-(Channel10-Pad13) -> Net-(JP1204-A)
- Channel10 pad 15: unconnected-(Channel10-Pad15) -> Net-(JP1205-A)
- Channel10 pad 9: unconnected-(Channel10-Pad9) -> Net-(JP1201-A)
- Channel11 pad 10: unconnected-(Channel11-Pad10) -> Net-(JP1502-A)
- Channel11 pad 11: unconnected-(Channel11-Pad11) -> Net-(JP1503-A)
- Channel11 pad 13: unconnected-(Channel11-Pad13) -> Net-(JP1504-A)
- Channel11 pad 15: unconnected-(Channel11-Pad15) -> Net-(JP1505-A)
- Channel11 pad 9: unconnected-(Channel11-Pad9) -> Net-(JP1501-A)
- Channel12 pad 10: unconnected-(Channel12-Pad10) -> Net-(JP1602-A)
- Channel12 pad 11: unconnected-(Channel12-Pad11) -> Net-(JP1603-A)
- Channel12 pad 13: unconnected-(Channel12-Pad13) -> Net-(JP1604-A)
- Channel12 pad 15: unconnected-(Channel12-Pad15) -> Net-(JP1605-A)
- Channel12 pad 9: unconnected-(Channel12-Pad9) -> Net-(JP1601-A)
- Channel13 pad 10: unconnected-(Channel13-Pad10) -> Net-(JP1702-A)
- Channel13 pad 11: unconnected-(Channel13-Pad11) -> Net-(JP1703-A)
- Channel13 pad 13: unconnected-(Channel13-Pad13) -> Net-(JP1704-A)
- Channel13 pad 15: unconnected-(Channel13-Pad15) -> Net-(JP1705-A)
- Channel13 pad 9: unconnected-(Channel13-Pad9) -> Net-(JP1701-A)
- Channel14 pad 10: unconnected-(Channel14-Pad10) -> Net-(JP1902-A)
- Channel14 pad 11: unconnected-(Channel14-Pad11) -> Net-(JP1903-A)
- Channel14 pad 13: unconnected-(Channel14-Pad13) -> Net-(JP1904-A)
- Channel14 pad 15: unconnected-(Channel14-Pad15) -> Net-(JP1905-A)
- Channel14 pad 9: unconnected-(Channel14-Pad9) -> Net-(JP1901-A)
- Channel15 pad 10: unconnected-(Channel15-Pad10) -> Net-(JP2002-A)
- Channel15 pad 11: unconnected-(Channel15-Pad11) -> Net-(JP2003-A)
- Channel15 pad 13: unconnected-(Channel15-Pad13) -> Net-(JP2004-A)
- Channel15 pad 15: unconnected-(Channel15-Pad15) -> Net-(JP2005-A)
- Channel15 pad 9: unconnected-(Channel15-Pad9) -> Net-(JP2001-A)
- Channel2 pad 10: unconnected-(Channel2-Pad10) -> Net-(JP302-A)
- Channel2 pad 11: unconnected-(Channel2-Pad11) -> Net-(JP303-A)
- Channel2 pad 13: unconnected-(Channel2-Pad13) -> Net-(JP304-A)
- Channel2 pad 15: unconnected-(Channel2-Pad15) -> Net-(JP305-A)
- Channel2 pad 9: unconnected-(Channel2-Pad9) -> Net-(JP301-A)
- Channel3 pad 10: unconnected-(Channel3-Pad10) -> Net-(JP402-A)
- Channel3 pad 11: unconnected-(Channel3-Pad11) -> Net-(JP403-A)
- Channel3 pad 13: unconnected-(Channel3-Pad13) -> Net-(JP404-A)
- Channel3 pad 15: unconnected-(Channel3-Pad15) -> Net-(JP405-A)
- Channel3 pad 9: unconnected-(Channel3-Pad9) -> Net-(JP401-A)
- Channel4 pad 10: unconnected-(Channel4-Pad10) -> Net-(JP502-A)
- Channel4 pad 11: unconnected-(Channel4-Pad11) -> Net-(JP503-A)
- Channel4 pad 13: unconnected-(Channel4-Pad13) -> Net-(JP504-A)
- Channel4 pad 15: unconnected-(Channel4-Pad15) -> Net-(JP505-A)
- Channel4 pad 9: unconnected-(Channel4-Pad9) -> Net-(JP501-A)
- Channel5 pad 10: unconnected-(Channel5-Pad10) -> Net-(JP602-A)
- Channel5 pad 11: unconnected-(Channel5-Pad11) -> Net-(JP603-A)
- Channel5 pad 13: unconnected-(Channel5-Pad13) -> Net-(JP604-A)
- Channel5 pad 15: unconnected-(Channel5-Pad15) -> Net-(JP605-A)
- Channel5 pad 9: unconnected-(Channel5-Pad9) -> Net-(JP601-A)
- Channel6 pad 10: unconnected-(Channel6-Pad10) -> Net-(JP702-A)
- Channel6 pad 11: unconnected-(Channel6-Pad11) -> Net-(JP703-A)
- Channel6 pad 13: unconnected-(Channel6-Pad13) -> Net-(JP704-A)
- Channel6 pad 15: unconnected-(Channel6-Pad15) -> Net-(JP705-A)
- Channel6 pad 9: unconnected-(Channel6-Pad9) -> Net-(JP701-A)
- Channel7 pad 10: unconnected-(Channel7-Pad10) -> Net-(JP802-A)
- Channel7 pad 11: unconnected-(Channel7-Pad11) -> Net-(JP803-A)
- Channel7 pad 13: unconnected-(Channel7-Pad13) -> Net-(JP804-A)
- Channel7 pad 15: unconnected-(Channel7-Pad15) -> Net-(JP805-A)
- Channel7 pad 9: unconnected-(Channel7-Pad9) -> Net-(JP801-A)
- Channel8 pad 10: unconnected-(Channel8-Pad10) -> Net-(JP902-A)
- Channel8 pad 11: unconnected-(Channel8-Pad11) -> Net-(JP903-A)
- Channel8 pad 13: unconnected-(Channel8-Pad13) -> Net-(JP904-A)
- Channel8 pad 15: unconnected-(Channel8-Pad15) -> Net-(JP905-A)
- Channel8 pad 9: unconnected-(Channel8-Pad9) -> Net-(JP901-A)
- Channel9 pad 10: unconnected-(Channel9-Pad10) -> Net-(JP1002-A)
- Channel9 pad 11: unconnected-(Channel9-Pad11) -> Net-(JP1003-A)
- Channel9 pad 13: unconnected-(Channel9-Pad13) -> Net-(JP1004-A)
- Channel9 pad 15: unconnected-(Channel9-Pad15) -> Net-(JP1005-A)
- Channel9 pad 9: unconnected-(Channel9-Pad9) -> Net-(JP1001-A)
Routing:
- net Net-(JP505-A): track 0.00 -> 9.12 mm, vias 0 -> 1
- net Net-(JP405-A): track 0.00 -> 9.12 mm, vias 0 -> 1
- net Net-(JP305-A): track 0.00 -> 9.12 mm, vias 0 -> 1
- net Net-(JP202-A): track 0.00 -> 9.12 mm, vias 0 -> 1
- net Net-(JP1802-A): track 0.00 -> 9.12 mm, vias 0 -> 1
- net Net-(JP805-A): track 0.00 -> 9.12 mm, vias 0 -> 1
- net Net-(JP802-A): track 0.00 -> 9.12 mm, vias 0 -> 1
- net Net-(JP705-A): track 0.00 -> 9.12 mm, vias 0 -> 1
- net Net-(JP702-A): track 0.00 -> 9.12 mm, vias 0 -> 1
- net Net-(JP605-A): track 0.00 -> 9.12 mm, vias 0 -> 1
- net Net-(JP602-A): track 0.00 -> 9.12 mm, vias 0 -> 1
- net Net-(JP502-A): track 0.00 -> 9.12 mm, vias 0 -> 1
- net Net-(JP402-A): track 0.00 -> 9.12 mm, vias 0 -> 1
- net Net-(JP302-A): track 0.00 -> 9.12 mm, vias 0 -> 1
- net Net-(JP205-A): track 0.00 -> 9.12 mm, vias 0 -> 1
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Other:
- board text added: "FEAR-16v2.2"
- board text removed: "FEAR-16v2.1"
