File: FEAR-16 - Mainboard.kicad_sch (KiCad schematic)
At the start: 50 parts, among them IC101 EK-TM4C123GXL, J101 Screw_5.08, U101 FT232RL, U102 SN74LVC1G14DBV, U103 SN74LVC1G14DBV, U104 HCPL-2631, U105 HCPL-2631, U106 SN74LVC1G14DBV, U107 SN74LVC1G14DBV

Commit message: Fixed ADP2370 designator
ADP2370 has a bunch of fixed output voltages and an adjustable model.
We use the adjustable model, so we fixed the name matching with the correct model-name.
Other:
- note added: "Schmitt-Trigger-Inverter: - SN74LVC1G14 - NC7S14M5X"

Commit message: Finished README.md
- Adjustment in .gitignore
- Finished first README.md attempt
- Added extra comments to "5V_Supplies"
Other:
- note added: "Schmitt-Trigger-Inverter: - SN74LVC1G14 - NC7S14M5X (alternative)"
- note removed: "Schmitt-Trigger-Inverter: - SN74LVC1G14 - NC7S14M5X"
Changed lines of the file:
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@@
 		)
 	)
-	(text "Schmitt-Trigger-Inverter:\n- SN74LVC1G14\n- NC7S14M5X"
+	(text "Schmitt-Trigger-Inverter:\n- SN74LVC1G14\n- NC7S14M5X (alternative)"
 		(exclude_from_sim no)
 		(at 93.89 186.97 0)
